File: simdir/simdir/simdir.kicad_pcb (KiCad board)
At the start: 4 copper layers, 240 x 139.8 mm, 84 parts, among them J1 Conn_Coaxial, Q1 BC847, Q10 BC847, Q11 BC847, Q12 BC847, Q13 BC847, Q14 BC847, Q15 BC847, Q16 BC847, Q2 BC847, Q3 BC847, Q4 BC847, Q5 BC847, Q6 BC847, Q7 BC847, Q8 BC847, Q9 BC847, U1 MASWSS0178, U10 MASWSS0178, U11 MASWSS0178, U12 MASWSS0178, U13 MASWSS0178, U14 MASWSS0178, U15 MASWSS0178, U16 MASWSS0178, U17 LTV-847S, U18 LTV-847S, U19 74HCT595, U2 MASWSS0178, U3 MASWSS0178, U4 MASWSS0178, U5 MASWSS0178, U6 MASWSS0178, U7 MASWSS0178, U8 MASWSS0178, U9 MASWSS0178

Commit message: Fixed minor issues with channel pins.
Connections:
- net /channel1/Dig_GND renamed /channel1/DIG_GND
- net /channel1/VCC renamed Net-(C1-Pad1)

Commit message: Duplicated the channels.
Parts:
- added C3: 470n, Capacitor_SMD:C_0805_2012Metric_Pad1.18x1.45mm_HandSolder, B.Cu at (252.7, 124.1)
- added C4: 470n, Capacitor_SMD:C_0805_2012Metric_Pad1.18x1.45mm_HandSolder, B.Cu at (192.9, 141.4)
- added C5: 470n, Capacitor_SMD:C_0805_2012Metric_Pad1.18x1.45mm_HandSolder, B.Cu at (252.7, 74.8)
- added C6: 470n, Capacitor_SMD:C_0805_2012Metric_Pad1.18x1.45mm_HandSolder, B.Cu at (193.0, 92.1)
- added FB2: FerriteBead, Inductor_SMD:L_0805_2012Metric_Pad1.05x1.20mm_HandSolder, B.Cu at (197.6, 141.4)
- added FB3: FerriteBead, Inductor_SMD:L_0805_2012Metric_Pad1.05x1.20mm_HandSolder, B.Cu at (197.6, 92.1)
- added J2: Conn_Coaxial, Connector_Coaxial:SMA_Amphenol_132289_EdgeMount, F.Cu at (23.3, 133.3)
- added J3: Conn_Coaxial, Connector_Coaxial:SMA_Amphenol_132289_EdgeMount, F.Cu at (23.3, 84.0)
- added Q17: BC847, Package_TO_SOT_SMD:SOT-23, B.Cu at (231.0, 99.6)
- added Q18: BC847, Package_TO_SOT_SMD:SOT-23, B.Cu at (231.1, 104.4)
- added Q19: BC847, Package_TO_SOT_SMD:SOT-23, B.Cu at (230.7, 109.6)
- added Q20: BC847, Package_TO_SOT_SMD:SOT-23, B.Cu at (230.5, 114.8)
- added Q21: BC847, Package_TO_SOT_SMD:SOT-23, B.Cu at (230.2, 120.6)
- added Q22: BC847, Package_TO_SOT_SMD:SOT-23, B.Cu at (230.2, 125.4)
- added Q23: BC847, Package_TO_SOT_SMD:SOT-23, B.Cu at (230.4, 130.6)
- added Q24: BC847, Package_TO_SOT_SMD:SOT-23, B.Cu at (230.5, 135.7)
- added Q25: BC847, Package_TO_SOT_SMD:SOT-23, B.Cu at (60.1, 133.1)
- added Q26: BC847, Package_TO_SOT_SMD:SOT-23, B.Cu at (71.2, 133.2)
- added Q27: BC847, Package_TO_SOT_SMD:SOT-23, B.Cu at (84.6, 133.1)
- added Q28: BC847, Package_TO_SOT_SMD:SOT-23, B.Cu at (100.1, 133.1)
- added Q29: BC847, Package_TO_SOT_SMD:SOT-23, B.Cu at (117.6, 133.1)
- added Q30: BC847, Package_TO_SOT_SMD:SOT-23, B.Cu at (134.9, 133.1)
- added Q31: BC847, Package_TO_SOT_SMD:SOT-23, B.Cu at (150.9, 133.1)
- added Q32: BC847, Package_TO_SOT_SMD:SOT-23, B.Cu at (167.4, 133.1)
- added Q33: BC847, Package_TO_SOT_SMD:SOT-23, B.Cu at (231.0, 50.3)
- added Q34: BC847, Package_TO_SOT_SMD:SOT-23, B.Cu at (231.2, 55.1)
- added Q35: BC847, Package_TO_SOT_SMD:SOT-23, B.Cu at (230.8, 60.3)
- added Q36: BC847, Package_TO_SOT_SMD:SOT-23, B.Cu at (230.6, 65.5)
- added Q37: BC847, Package_TO_SOT_SMD:SOT-23, B.Cu at (230.3, 71.3)
- added Q38: BC847, Package_TO_SOT_SMD:SOT-23, B.Cu at (230.3, 76.1)
- added Q39: BC847, Package_TO_SOT_SMD:SOT-23, B.Cu at (230.4, 81.3)
- added Q40: BC847, Package_TO_SOT_SMD:SOT-23, B.Cu at (230.5, 86.4)
- added Q41: BC847, Package_TO_SOT_SMD:SOT-23, B.Cu at (60.2, 83.8)
- added Q42: BC847, Package_TO_SOT_SMD:SOT-23, B.Cu at (71.2, 83.9)
- added Q43: BC847, Package_TO_SOT_SMD:SOT-23, B.Cu at (84.7, 83.8)
- added Q44: BC847, Package_TO_SOT_SMD:SOT-23, B.Cu at (100.2, 83.8)
- added Q45: BC847, Package_TO_SOT_SMD:SOT-23, B.Cu at (117.7, 83.8)
- added Q46: BC847, Package_TO_SOT_SMD:SOT-23, B.Cu at (134.9, 83.8)
- added Q47: BC847, Package_TO_SOT_SMD:SOT-23, B.Cu at (150.9, 83.8)
- added Q48: BC847, Package_TO_SOT_SMD:SOT-23, B.Cu at (167.4, 83.8)
- added R100: 1k, Resistor_SMD:R_0805_2012Metric_Pad1.20x1.40mm_HandSolder, B.Cu at (208.0, 78.8)
- added R101: 1k, Resistor_SMD:R_0805_2012Metric_Pad1.20x1.40mm_HandSolder, B.Cu at (207.7, 83.8)
- added R102: 1k, Resistor_SMD:R_0805_2012Metric_Pad1.20x1.40mm_HandSolder, B.Cu at (207.7, 88.8)
- added R103: 10k, Resistor_SMD:R_0805_2012Metric_Pad1.20x1.40mm_HandSolder, B.Cu at (64.0, 89.1)
- added R104: 10k, Resistor_SMD:R_0805_2012Metric_Pad1.20x1.40mm_HandSolder, B.Cu at (76.5, 89.1)
- added R105: 10k, Resistor_SMD:R_0805_2012Metric_Pad1.20x1.40mm_HandSolder, B.Cu at (90.0, 89.1)
- added R106: 10k, Resistor_SMD:R_0805_2012Metric_Pad1.20x1.40mm_HandSolder, B.Cu at (106.7, 89.1)
- added R107: 100k, Resistor_SMD:R_0805_2012Metric_Pad1.20x1.40mm_HandSolder, B.Cu at (64.0, 83.8)
- added R108: 100k, Resistor_SMD:R_0805_2012Metric_Pad1.20x1.40mm_HandSolder, B.Cu at (76.5, 83.8)
- added R109: 100k, Resistor_SMD:R_0805_2012Metric_Pad1.20x1.40mm_HandSolder, B.Cu at (90.0, 83.8)
- added R110: 100k, Resistor_SMD:R_0805_2012Metric_Pad1.20x1.40mm_HandSolder, B.Cu at (106.7, 83.8)
- added R111: 10k, Resistor_SMD:R_0805_2012Metric_Pad1.20x1.40mm_HandSolder, B.Cu at (60.2, 89.1)
- added R112: 10k, Resistor_SMD:R_0805_2012Metric_Pad1.20x1.40mm_HandSolder, B.Cu at (71.2, 89.1)
- added R113: 10k, Resistor_SMD:R_0805_2012Metric_Pad1.20x1.40mm_HandSolder, B.Cu at (84.7, 89.1)
- added R114: 10k, Resistor_SMD:R_0805_2012Metric_Pad1.20x1.40mm_HandSolder, B.Cu at (100.2, 89.1)
- added R115: 10k, Resistor_SMD:R_0805_2012Metric_Pad1.20x1.40mm_HandSolder, B.Cu at (125.2, 88.8)
- added R116: 10k, Resistor_SMD:R_0805_2012Metric_Pad1.20x1.40mm_HandSolder, B.Cu at (140.0, 89.1)
- added R117: 10k, Resistor_SMD:R_0805_2012Metric_Pad1.20x1.40mm_HandSolder, B.Cu at (157.7, 89.1)
- added R118: 10k, Resistor_SMD:R_0805_2012Metric_Pad1.20x1.40mm_HandSolder, B.Cu at (175.2, 89.1)
- added R119: 63.4, Resistor_SMD:R_0805_2012Metric_Pad1.20x1.40mm_HandSolder, F.Cu at (35.0, 82.1)
- added R120: 100k, Resistor_SMD:R_0805_2012Metric_Pad1.20x1.40mm_HandSolder, B.Cu at (125.2, 83.6)
- added R121: 100k, Resistor_SMD:R_0805_2012Metric_Pad1.20x1.40mm_HandSolder, B.Cu at (140.0, 83.8)
- added R122: 100k, Resistor_SMD:R_0805_2012Metric_Pad1.20x1.40mm_HandSolder, B.Cu at (157.7, 83.8)
- added R123: 100k, Resistor_SMD:R_0805_2012Metric_Pad1.20x1.40mm_HandSolder, B.Cu at (175.2, 83.8)
- added R124: 71.5, Resistor_SMD:R_0805_2012Metric_Pad1.20x1.40mm_HandSolder, F.Cu at (30.7, 80.8)
- added R125: 63.4, Resistor_SMD:R_0805_2012Metric_Pad1.20x1.40mm_HandSolder, F.Cu at (30.7, 83.8)
- added R126: 10k, Resistor_SMD:R_0805_2012Metric_Pad1.20x1.40mm_HandSolder, B.Cu at (117.7, 89.1)
- added R127: 10k, Resistor_SMD:R_0805_2012Metric_Pad1.20x1.40mm_HandSolder, B.Cu at (135.0, 89.1)
- added R128: 10k, Resistor_SMD:R_0805_2012Metric_Pad1.20x1.40mm_HandSolder, B.Cu at (151.0, 89.1)
- added R129: 10k, Resistor_SMD:R_0805_2012Metric_Pad1.20x1.40mm_HandSolder, B.Cu at (167.5, 89.1)
- added R44: 10k, Resistor_SMD:R_0805_2012Metric_Pad1.20x1.40mm_HandSolder, B.Cu at (236.9, 98.6)
- added R45: 10k, Resistor_SMD:R_0805_2012Metric_Pad1.20x1.40mm_HandSolder, B.Cu at (236.7, 103.6)
- added R46: 10k, Resistor_SMD:R_0805_2012Metric_Pad1.20x1.40mm_HandSolder, B.Cu at (236.7, 108.6)
- added R47: 10k, Resistor_SMD:R_0805_2012Metric_Pad1.20x1.40mm_HandSolder, B.Cu at (236.7, 113.9)
- added R48: 1k, Resistor_SMD:R_0805_2012Metric_Pad1.20x1.40mm_HandSolder, B.Cu at (207.9, 99.4)
- added R49: 1k, Resistor_SMD:R_0805_2012Metric_Pad1.20x1.40mm_HandSolder, B.Cu at (207.9, 104.4)
- added R50: 1k, Resistor_SMD:R_0805_2012Metric_Pad1.20x1.40mm_HandSolder, B.Cu at (207.9, 109.6)
- added R51: 1k, Resistor_SMD:R_0805_2012Metric_Pad1.20x1.40mm_HandSolder, B.Cu at (207.9, 114.9)
- added R52: 10k, Resistor_SMD:R_0805_2012Metric_Pad1.20x1.40mm_HandSolder, B.Cu at (236.4, 119.6)
- added R53: 10k, Resistor_SMD:R_0805_2012Metric_Pad1.20x1.40mm_HandSolder, B.Cu at (236.4, 124.6)
- added R54: 10k, Resistor_SMD:R_0805_2012Metric_Pad1.20x1.40mm_HandSolder, B.Cu at (236.4, 129.6)
- added R55: 10k, Resistor_SMD:R_0805_2012Metric_Pad1.20x1.40mm_HandSolder, B.Cu at (236.4, 134.6)
- added R56: 1k, Resistor_SMD:R_0805_2012Metric_Pad1.20x1.40mm_HandSolder, B.Cu at (207.9, 123.1)
- added R57: 1k, Resistor_SMD:R_0805_2012Metric_Pad1.20x1.40mm_HandSolder, B.Cu at (207.9, 128.1)
- added R58: 1k, Resistor_SMD:R_0805_2012Metric_Pad1.20x1.40mm_HandSolder, B.Cu at (207.7, 133.1)
- added R59: 1k, Resistor_SMD:R_0805_2012Metric_Pad1.20x1.40mm_HandSolder, B.Cu at (207.7, 138.1)
- added R60: 10k, Resistor_SMD:R_0805_2012Metric_Pad1.20x1.40mm_HandSolder, B.Cu at (63.9, 138.4)
- added R61: 10k, Resistor_SMD:R_0805_2012Metric_Pad1.20x1.40mm_HandSolder, B.Cu at (76.4, 138.4)
- added R62: 10k, Resistor_SMD:R_0805_2012Metric_Pad1.20x1.40mm_HandSolder, B.Cu at (89.9, 138.4)
- added R63: 10k, Resistor_SMD:R_0805_2012Metric_Pad1.20x1.40mm_HandSolder, B.Cu at (106.7, 138.4)
- added R64: 100k, Resistor_SMD:R_0805_2012Metric_Pad1.20x1.40mm_HandSolder, B.Cu at (63.9, 133.1)
- added R65: 100k, Resistor_SMD:R_0805_2012Metric_Pad1.20x1.40mm_HandSolder, B.Cu at (76.4, 133.1)
- added R66: 100k, Resistor_SMD:R_0805_2012Metric_Pad1.20x1.40mm_HandSolder, B.Cu at (89.9, 133.1)
- added R67: 100k, Resistor_SMD:R_0805_2012Metric_Pad1.20x1.40mm_HandSolder, B.Cu at (106.7, 133.1)
- added R68: 10k, Resistor_SMD:R_0805_2012Metric_Pad1.20x1.40mm_HandSolder, B.Cu at (60.2, 138.4)
- added R69: 10k, Resistor_SMD:R_0805_2012Metric_Pad1.20x1.40mm_HandSolder, B.Cu at (71.2, 138.4)
- added R70: 10k, Resistor_SMD:R_0805_2012Metric_Pad1.20x1.40mm_HandSolder, B.Cu at (84.7, 138.4)
- added R71: 10k, Resistor_SMD:R_0805_2012Metric_Pad1.20x1.40mm_HandSolder, B.Cu at (100.2, 138.4)
- added R72: 10k, Resistor_SMD:R_0805_2012Metric_Pad1.20x1.40mm_HandSolder, B.Cu at (125.2, 138.1)
- added R73: 10k, Resistor_SMD:R_0805_2012Metric_Pad1.20x1.40mm_HandSolder, B.Cu at (139.9, 138.4)
- added R74: 10k, Resistor_SMD:R_0805_2012Metric_Pad1.20x1.40mm_HandSolder, B.Cu at (157.7, 138.4)
- added R75: 10k, Resistor_SMD:R_0805_2012Metric_Pad1.20x1.40mm_HandSolder, B.Cu at (175.2, 138.4)
- added R76: 63.4, Resistor_SMD:R_0805_2012Metric_Pad1.20x1.40mm_HandSolder, F.Cu at (34.9, 131.4)
- added R77: 100k, Resistor_SMD:R_0805_2012Metric_Pad1.20x1.40mm_HandSolder, B.Cu at (125.2, 132.9)
- added R78: 100k, Resistor_SMD:R_0805_2012Metric_Pad1.20x1.40mm_HandSolder, B.Cu at (139.9, 133.1)
- added R79: 100k, Resistor_SMD:R_0805_2012Metric_Pad1.20x1.40mm_HandSolder, B.Cu at (157.7, 133.1)
- added R80: 100k, Resistor_SMD:R_0805_2012Metric_Pad1.20x1.40mm_HandSolder, B.Cu at (175.2, 133.1)
- added R81: 71.5, Resistor_SMD:R_0805_2012Metric_Pad1.20x1.40mm_HandSolder, F.Cu at (30.7, 130.1)
- added R82: 63.4, Resistor_SMD:R_0805_2012Metric_Pad1.20x1.40mm_HandSolder, F.Cu at (30.7, 133.1)
- added R83: 10k, Resistor_SMD:R_0805_2012Metric_Pad1.20x1.40mm_HandSolder, B.Cu at (117.7, 138.4)
- added R84: 10k, Resistor_SMD:R_0805_2012Metric_Pad1.20x1.40mm_HandSolder, B.Cu at (134.9, 138.4)
- added R85: 10k, Resistor_SMD:R_0805_2012Metric_Pad1.20x1.40mm_HandSolder, B.Cu at (150.9, 138.4)
- added R86: 10k, Resistor_SMD:R_0805_2012Metric_Pad1.20x1.40mm_HandSolder, B.Cu at (167.4, 138.4)
- added R87: 10k, Resistor_SMD:R_0805_2012Metric_Pad1.20x1.40mm_HandSolder, B.Cu at (237.0, 49.3)
- added R88: 10k, Resistor_SMD:R_0805_2012Metric_Pad1.20x1.40mm_HandSolder, B.Cu at (236.7, 54.3)
- added R89: 10k, Resistor_SMD:R_0805_2012Metric_Pad1.20x1.40mm_HandSolder, B.Cu at (236.7, 59.3)
- added R90: 10k, Resistor_SMD:R_0805_2012Metric_Pad1.20x1.40mm_HandSolder, B.Cu at (236.7, 64.6)
- added R91: 1k, Resistor_SMD:R_0805_2012Metric_Pad1.20x1.40mm_HandSolder, B.Cu at (208.0, 50.1)
- added R92: 1k, Resistor_SMD:R_0805_2012Metric_Pad1.20x1.40mm_HandSolder, B.Cu at (208.0, 55.1)
- added R93: 1k, Resistor_SMD:R_0805_2012Metric_Pad1.20x1.40mm_HandSolder, B.Cu at (208.0, 60.3)
- added R94: 1k, Resistor_SMD:R_0805_2012Metric_Pad1.20x1.40mm_HandSolder, B.Cu at (208.0, 65.6)
- added R95: 10k, Resistor_SMD:R_0805_2012Metric_Pad1.20x1.40mm_HandSolder, B.Cu at (236.5, 70.3)
- added R96: 10k, Resistor_SMD:R_0805_2012Metric_Pad1.20x1.40mm_HandSolder, B.Cu at (236.5, 75.3)
- added R97: 10k, Resistor_SMD:R_0805_2012Metric_Pad1.20x1.40mm_HandSolder, B.Cu at (236.5, 80.3)
- added R98: 10k, Resistor_SMD:R_0805_2012Metric_Pad1.20x1.40mm_HandSolder, B.Cu at (236.5, 85.3)
- added R99: 1k, Resistor_SMD:R_0805_2012Metric_Pad1.20x1.40mm_HandSolder, B.Cu at (208.0, 73.8)
- added SWLSB2: CTS221, hand:CTS221, F.Cu at (216.1, 110.3)
- added SWLSB3: CTS221, hand:CTS221, F.Cu at (216.2, 61.0)
- added SWMSB2: CTS221, hand:CTS221, F.Cu at (216.3, 120.5)
- added SWMSB3: CTS221, hand:CTS221, F.Cu at (216.4, 71.2)
- added U20: 74HCT595, Package_SO:SOIC-16_3.9x9.9mm_P1.27mm, B.Cu at (250.9, 116.6)
- added U21: MASWSS0178, hand:MSOP-8-1EP_3x3mm_P0.65mm_EP1.73x1.85mm_hand, F.Cu at (48.0, 108.4)
- added U22: MASWSS0178, hand:MSOP-8-1EP_3x3mm_P0.65mm_EP1.73x1.85mm_hand, F.Cu at (65.0, 108.4)
- added U23: MASWSS0178, hand:MSOP-8-1EP_3x3mm_P0.65mm_EP1.73x1.85mm_hand, F.Cu at (82.0, 108.4)
- added U24: MASWSS0178, hand:MSOP-8-1EP_3x3mm_P0.65mm_EP1.73x1.85mm_hand, F.Cu at (99.0, 108.4)
- added U25: LTV-847S, Package_DIP:SMDIP-16_W9.53mm, B.Cu at (197.7, 105.8)
- added U26: MASWSS0178, hand:MSOP-8-1EP_3x3mm_P0.65mm_EP1.73x1.85mm_hand, F.Cu at (90.0, 108.4)
- added U27: MASWSS0178, hand:MSOP-8-1EP_3x3mm_P0.65mm_EP1.73x1.85mm_hand, F.Cu at (107.0, 108.4)
- added U28: MASWSS0178, hand:MSOP-8-1EP_3x3mm_P0.65mm_EP1.73x1.85mm_hand, F.Cu at (56.0, 108.4)
- added U29: MASWSS0178, hand:MSOP-8-1EP_3x3mm_P0.65mm_EP1.73x1.85mm_hand, F.Cu at (73.1, 108.3)
- added U30: LTV-847S, Package_DIP:SMDIP-16_W9.53mm, B.Cu at (197.7, 129.3)
- added U31: MASWSS0178, hand:MSOP-8-1EP_3x3mm_P0.65mm_EP1.73x1.85mm_hand, F.Cu at (116.0, 108.4)
- added U32: MASWSS0178, hand:MSOP-8-1EP_3x3mm_P0.65mm_EP1.73x1.85mm_hand, F.Cu at (133.1, 108.3)
- added U33: MASWSS0178, hand:MSOP-8-1EP_3x3mm_P0.65mm_EP1.73x1.85mm_hand, F.Cu at (150.1, 108.3)
- added U34: MASWSS0178, hand:MSOP-8-1EP_3x3mm_P0.65mm_EP1.73x1.85mm_hand, F.Cu at (166.7, 108.3)
- added U35: MASWSS0178, hand:MSOP-8-1EP_3x3mm_P0.65mm_EP1.73x1.85mm_hand, F.Cu at (124.1, 108.3)
- added U36: MASWSS0178, hand:MSOP-8-1EP_3x3mm_P0.65mm_EP1.73x1.85mm_hand, F.Cu at (141.2, 108.3)
- added U37: MASWSS0178, hand:MSOP-8-1EP_3x3mm_P0.65mm_EP1.73x1.85mm_hand, F.Cu at (158.1, 108.4)
- added U38: MASWSS0178, hand:MSOP-8-1EP_3x3mm_P0.65mm_EP1.73x1.85mm_hand, F.Cu at (174.7, 108.3)
- added U39: 74HCT595, Package_SO:SOIC-16_3.9x9.9mm_P1.27mm, B.Cu at (251.0, 67.3)
- added U40: MASWSS0178, hand:MSOP-8-1EP_3x3mm_P0.65mm_EP1.73x1.85mm_hand, F.Cu at (48.0, 59.1)
- added U41: MASWSS0178, hand:MSOP-8-1EP_3x3mm_P0.65mm_EP1.73x1.85mm_hand, F.Cu at (65.0, 59.1)
- added U42: MASWSS0178, hand:MSOP-8-1EP_3x3mm_P0.65mm_EP1.73x1.85mm_hand, F.Cu at (82.0, 59.1)
- added U43: MASWSS0178, hand:MSOP-8-1EP_3x3mm_P0.65mm_EP1.73x1.85mm_hand, F.Cu at (99.0, 59.1)
- added U44: LTV-847S, Package_DIP:SMDIP-16_W9.53mm, B.Cu at (197.7, 56.5)
- added U45: MASWSS0178, hand:MSOP-8-1EP_3x3mm_P0.65mm_EP1.73x1.85mm_hand, F.Cu at (90.0, 59.1)
- added U46: MASWSS0178, hand:MSOP-8-1EP_3x3mm_P0.65mm_EP1.73x1.85mm_hand, F.Cu at (107.0, 59.1)
- added U47: MASWSS0178, hand:MSOP-8-1EP_3x3mm_P0.65mm_EP1.73x1.85mm_hand, F.Cu at (56.0, 59.1)
- added U48: MASWSS0178, hand:MSOP-8-1EP_3x3mm_P0.65mm_EP1.73x1.85mm_hand, F.Cu at (73.1, 59.0)
- added U49: LTV-847S, Package_DIP:SMDIP-16_W9.53mm, B.Cu at (197.7, 80.0)
- added U50: MASWSS0178, hand:MSOP-8-1EP_3x3mm_P0.65mm_EP1.73x1.85mm_hand, F.Cu at (116.0, 59.1)
- added U51: MASWSS0178, hand:MSOP-8-1EP_3x3mm_P0.65mm_EP1.73x1.85mm_hand, F.Cu at (133.1, 59.0)
- added U52: MASWSS0178, hand:MSOP-8-1EP_3x3mm_P0.65mm_EP1.73x1.85mm_hand, F.Cu at (150.1, 59.0)
- added U53: MASWSS0178, hand:MSOP-8-1EP_3x3mm_P0.65mm_EP1.73x1.85mm_hand, F.Cu at (166.8, 59.0)
- added U54: MASWSS0178, hand:MSOP-8-1EP_3x3mm_P0.65mm_EP1.73x1.85mm_hand, F.Cu at (124.1, 59.0)
- added U55: MASWSS0178, hand:MSOP-8-1EP_3x3mm_P0.65mm_EP1.73x1.85mm_hand, F.Cu at (141.3, 59.0)
- added U56: MASWSS0178, hand:MSOP-8-1EP_3x3mm_P0.65mm_EP1.73x1.85mm_hand, F.Cu at (158.1, 59.1)
- added U57: MASWSS0178, hand:MSOP-8-1EP_3x3mm_P0.65mm_EP1.73x1.85mm_hand, F.Cu at (174.8, 59.0)
- moved Q10 33.3 mm to (230.9, 153.3)
- moved SWLSB1 33.3 mm to (215.9, 159.2)
- moved U4 33.3 mm to (98.8, 157.2)
- moved U7 33.3 mm to (89.8, 157.2)
- moved U8 33.3 mm to (106.8, 157.2)
- moved U9 33.3 mm to (115.8, 157.2)
- moved C1 33.3 mm to (192.8, 190.2)
- moved C2 33.3 mm to (252.5, 173.0)
- moved FB1 33.3 mm to (197.4, 190.2)
- moved J1 33.3 mm to (23.1, 182.1)
- moved Q1 33.3 mm to (60.0, 181.9)
- moved Q12 33.3 mm to (230.4, 163.7)
- moved Q13 33.3 mm to (230.1, 169.4)
- moved Q14 33.3 mm to (230.1, 174.3)
- moved Q15 33.3 mm to (230.2, 179.5)
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Routing:
- net /channel3/RF0_meander: track 0.00 -> 677.0 mm
- net /channel2/RF0_meander: track 0.00 -> 677.0 mm
- net /channel3/RF7_meander: track 0.00 -> 340.9 mm
- net /channel2/RF7_meander: track 0.00 -> 340.9 mm
- net Net-(U41-CTL1): track 0.00 -> 286.4 mm, vias 0 -> 2
- net Net-(U22-CTL1): track 0.00 -> 286.4 mm, vias 0 -> 2
- net Net-(U40-CTL1): track 0.00 -> 260.8 mm, vias 0 -> 3
- net Net-(U21-CTL1): track 0.00 -> 260.8 mm, vias 0 -> 3
- net /channel3/RF_GND: track 0.00 -> 199.7 mm, vias 0 -> 177
- net /channel2/RF_GND: track 0.00 -> 199.7 mm, vias 0 -> 177
- net Net-(U57-RFC): track 0.00 -> 192.3 mm
- net Net-(U38-RFC): track 0.00 -> 192.3 mm
- net /channel2/RF1_meander: track 0.00 -> 170.8 mm
- net /channel3/RF1_meander: track 0.00 -> 170.8 mm
- net Net-(U42-CTL1): track 0.00 -> 164.2 mm, vias 0 -> 2
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- added copper zone on B.Cu, net /channel2/5v
- added copper zone on F.Cu, net /channel2/RF_GND
- added copper zone on B.Cu, net /channel3/5v
- added copper zone on F.Cu, net /channel3/RF_GND
Other:
- board size 240 x 139.8 mm -> 240 x 177.2 mm
- board text added: "East"
- board text added: "North"
- board text added: "West"

Commit message: Fixed layout issues & added splitter.
Parts:
- added J4: Conn_02x05_Odd_Even, Connector_PinHeader_2.54mm:PinHeader_2x05_P2.54mm_Vertical, F.Cu at (220.6, -10.6)
- added J5: Conn_Coaxial, Connector_Coaxial:SMA_Amphenol_132289_EdgeMount, F.Cu at (29.4, 44.0)
- added R130: 10k, Resistor_SMD:R_0805_2012Metric_Pad1.20x1.40mm_HandSolder, F.Cu at (228.6, -22.5)
- added R131: 24.9, Resistor_SMD:R_0805_2012Metric_Pad1.20x1.40mm_HandSolder, F.Cu at (41.0, 44.0)
- added R132: 24.9, Resistor_SMD:R_0805_2012Metric_Pad1.20x1.40mm_HandSolder, F.Cu at (40.9, 46.8)
- added R133: 24.9, Resistor_SMD:R_0805_2012Metric_Pad1.20x1.40mm_HandSolder, F.Cu at (40.9, 41.0)
- moved J3 7.46 mm to (29.2, 79.4)
- moved R119 7.11 mm to (36.1, 75.0), turned to -90 degrees
- moved J2 7.09 mm to (29.6, 130.1)
- moved J1 6.42 mm to (29.4, 180.9)
- moved R41 6.36 mm to (36.0, 185.2), turned to 90 degrees
- moved R76 5.80 mm to (36.5, 125.8), turned to -90 degrees
- moved C5 5.75 mm to (257.4, 71.5)
- moved C6 5.75 mm to (197.6, 88.7)
- moved Q36 5.75 mm to (235.3, 62.2)
- moved Q37 5.75 mm to (235.0, 67.9)
- moved Q39 5.75 mm to (235.1, 78.0)
- moved R100 5.75 mm to (212.6, 75.5)
- moved R101 5.75 mm to (212.4, 80.5)
- moved R102 5.75 mm to (212.4, 85.5)
- moved R95 5.75 mm to (241.1, 67.0)
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Connections:
- C1 pad 2: /channel1/RF_GND -> RF_GND
- C2 pad 1: /channel1/5v -> 5v
- C2 pad 2: /channel1/DIG_GND -> DIG_GND
- C3 pad 1: /channel2/5v -> 5v
- C3 pad 2: /channel2/DIG_GND -> DIG_GND
- C4 pad 2: /channel2/RF_GND -> RF_GND
- C5 pad 1: /channel3/5v -> 5v
- C5 pad 2: /channel3/DIG_GND -> DIG_GND
- C6 pad 2: /channel3/RF_GND -> RF_GND
- FB1 pad 1: /channel1/5v -> 5v
- FB2 pad 1: /channel2/5v -> 5v
- FB3 pad 1: /channel3/5v -> 5v
- J1 pad 2: /channel1/RF_GND -> RF_GND
- J2 pad 2: /channel2/RF_GND -> RF_GND
- J3 pad 2: /channel3/RF_GND -> RF_GND
- Q1 pad 2: /channel1/RF_GND -> RF_GND
- Q10 pad 2: /channel1/DIG_GND -> DIG_GND
- Q11 pad 2: /channel1/DIG_GND -> DIG_GND
- Q12 pad 2: /channel1/DIG_GND -> DIG_GND
- Q13 pad 2: /channel1/DIG_GND -> DIG_GND
- Q14 pad 2: /channel1/DIG_GND -> DIG_GND
- Q15 pad 2: /channel1/DIG_GND -> DIG_GND
- Q16 pad 2: /channel1/DIG_GND -> DIG_GND
- Q17 pad 2: /channel2/DIG_GND -> DIG_GND
- Q18 pad 2: /channel2/DIG_GND -> DIG_GND
- Q19 pad 2: /channel2/DIG_GND -> DIG_GND
- Q2 pad 2: /channel1/RF_GND -> RF_GND
- Q20 pad 2: /channel2/DIG_GND -> DIG_GND
- Q21 pad 2: /channel2/DIG_GND -> DIG_GND
- Q22 pad 2: /channel2/DIG_GND -> DIG_GND
- Q23 pad 2: /channel2/DIG_GND -> DIG_GND
- Q24 pad 2: /channel2/DIG_GND -> DIG_GND
- Q25 pad 2: /channel2/RF_GND -> RF_GND
- Q26 pad 2: /channel2/RF_GND -> RF_GND
- Q27 pad 2: /channel2/RF_GND -> RF_GND
- Q28 pad 2: /channel2/RF_GND -> RF_GND
- Q29 pad 2: /channel2/RF_GND -> RF_GND
- Q3 pad 2: /channel1/RF_GND -> RF_GND
- Q30 pad 2: /channel2/RF_GND -> RF_GND
- Q31 pad 2: /channel2/RF_GND -> RF_GND
- Q32 pad 2: /channel2/RF_GND -> RF_GND
- Q33 pad 2: /channel3/DIG_GND -> DIG_GND
- Q34 pad 2: /channel3/DIG_GND -> DIG_GND
- Q35 pad 2: /channel3/DIG_GND -> DIG_GND
- Q36 pad 2: /channel3/DIG_GND -> DIG_GND
- Q37 pad 2: /channel3/DIG_GND -> DIG_GND
- Q38 pad 2: /channel3/DIG_GND -> DIG_GND
- Q39 pad 2: /channel3/DIG_GND -> DIG_GND
- Q4 pad 2: /channel1/RF_GND -> RF_GND
- Q40 pad 2: /channel3/DIG_GND -> DIG_GND
- Q41 pad 2: /channel3/RF_GND -> RF_GND
- Q42 pad 2: /channel3/RF_GND -> RF_GND
- Q43 pad 2: /channel3/RF_GND -> RF_GND
- Q44 pad 2: /channel3/RF_GND -> RF_GND
- Q45 pad 2: /channel3/RF_GND -> RF_GND
- Q46 pad 2: /channel3/RF_GND -> RF_GND
- Q47 pad 2: /channel3/RF_GND -> RF_GND
- Q48 pad 2: /channel3/RF_GND -> RF_GND
- Q5 pad 2: /channel1/RF_GND -> RF_GND
- Q6 pad 2: /channel1/RF_GND -> RF_GND
- Q7 pad 2: /channel1/RF_GND -> RF_GND
- Q8 pad 2: /channel1/RF_GND -> RF_GND
- Q9 pad 2: /channel1/DIG_GND -> DIG_GND
- R119 pad 1: /channel3/RF_GND -> RF_GND
- R119 pad 2: Net-(U57-RFC) -> Net-(J3-In)
- R124 pad 1: Net-(J3-In) -> Net-(U40-RFC)
- R124 pad 2: Net-(U57-RFC) -> Net-(J3-In)
- R125 pad 1: /channel3/RF_GND -> RF_GND
- R125 pad 2: Net-(J3-In) -> Net-(U40-RFC)
- R41 pad 1: /channel1/RF_GND -> RF_GND
- R41 pad 2: Net-(J1-In) -> Net-(U1-RFC)
- R42 pad 1: /channel1/RF_GND -> RF_GND
- R42 pad 2: Net-(U16-RFC) -> Net-(J1-In)
- R43 pad 1: Net-(J1-In) -> Net-(U1-RFC)
- R43 pad 2: Net-(U16-RFC) -> Net-(J1-In)
- R76 pad 1: /channel2/RF_GND -> RF_GND
- R76 pad 2: Net-(U38-RFC) -> Net-(J2-In)
- R81 pad 1: Net-(J2-In) -> Net-(U21-RFC)
- R81 pad 2: Net-(U38-RFC) -> Net-(J2-In)
- R82 pad 1: /channel2/RF_GND -> RF_GND
- R82 pad 2: Net-(J2-In) -> Net-(U21-RFC)
- SWLSB1 pad 2: /channel1/DIG_GND -> DIG_GND
- SWLSB1 pad 5: /channel1/DIG_GND -> DIG_GND
- SWLSB2 pad 2: /channel2/DIG_GND -> DIG_GND
- SWLSB2 pad 5: /channel2/DIG_GND -> DIG_GND
- SWLSB3 pad 2: /channel3/DIG_GND -> DIG_GND
- SWLSB3 pad 5: /channel3/DIG_GND -> DIG_GND
- SWMSB1 pad 2: /channel1/DIG_GND -> DIG_GND
- SWMSB1 pad 5: /channel1/DIG_GND -> DIG_GND
- SWMSB2 pad 2: /channel2/DIG_GND -> DIG_GND
- SWMSB2 pad 5: /channel2/DIG_GND -> DIG_GND
- SWMSB3 pad 2: /channel3/DIG_GND -> DIG_GND
- SWMSB3 pad 5: /channel3/DIG_GND -> DIG_GND
- U1 pad 3: /channel1/RF-In -> Net-(U1-RFC)
- U1 pad 4: /channel1/RF_GND -> RF_GND
- U1 pad 6: /channel1/RF_GND -> RF_GND
- U1 pad 7: /channel1/RF_GND -> RF_GND
- U1 pad 9: /channel1/RF_GND -> RF_GND
- U10 pad 4: /channel1/RF_GND -> RF_GND
- U10 pad 6: /channel1/RF_GND -> RF_GND
- U10 pad 7: /channel1/RF_GND -> RF_GND
- U10 pad 9: /channel1/RF_GND -> RF_GND
- U11 pad 4: /channel1/RF_GND -> RF_GND
- U11 pad 6: /channel1/RF_GND -> RF_GND
- U11 pad 7: /channel1/RF_GND -> RF_GND
- U11 pad 9: /channel1/RF_GND -> RF_GND
- U12 pad 4: /channel1/RF_GND -> RF_GND
- U12 pad 6: /channel1/RF_GND -> RF_GND
- U12 pad 7: /channel1/RF_GND -> RF_GND
- U12 pad 9: /channel1/RF_GND -> RF_GND
- U13 pad 4: /channel1/RF_GND -> RF_GND
- U13 pad 6: /channel1/RF_GND -> RF_GND
- U13 pad 7: /channel1/RF_GND -> RF_GND
- U13 pad 9: /channel1/RF_GND -> RF_GND
- U14 pad 4: /channel1/RF_GND -> RF_GND
- U14 pad 6: /channel1/RF_GND -> RF_GND
- U14 pad 7: /channel1/RF_GND -> RF_GND
- U14 pad 9: /channel1/RF_GND -> RF_GND
- U15 pad 4: /channel1/RF_GND -> RF_GND
- U15 pad 6: /channel1/RF_GND -> RF_GND
- U15 pad 7: /channel1/RF_GND -> RF_GND
- U15 pad 9: /channel1/RF_GND -> RF_GND
- U16 pad 3: Net-(U16-RFC) -> /channel1/RF-In
- U16 pad 4: /channel1/RF_GND -> RF_GND
- U16 pad 6: /channel1/RF_GND -> RF_GND
- U16 pad 7: /channel1/RF_GND -> RF_GND
- U16 pad 9: /channel1/RF_GND -> RF_GND
- U17 pad 1: /channel1/5v -> 5v
- U17 pad 11: /channel1/RF_GND -> RF_GND
- U17 pad 13: /channel1/RF_GND -> RF_GND
- U17 pad 15: /channel1/RF_GND -> RF_GND
- U17 pad 3: /channel1/5v -> 5v
- U17 pad 5: /channel1/5v -> 5v
- U17 pad 7: /channel1/5v -> 5v
- U17 pad 9: /channel1/RF_GND -> RF_GND
- U18 pad 1: /channel1/5v -> 5v
- U18 pad 11: /channel1/RF_GND -> RF_GND
- U18 pad 13: /channel1/RF_GND -> RF_GND
- U18 pad 15: /channel1/RF_GND -> RF_GND
- U18 pad 3: /channel1/5v -> 5v
- U18 pad 5: /channel1/5v -> 5v
- U18 pad 7: /channel1/5v -> 5v
- U18 pad 9: /channel1/RF_GND -> RF_GND
- U19 pad 16: /channel1/5v -> 5v
- U19 pad 8: /channel1/DIG_GND -> DIG_GND
- U2 pad 4: /channel1/RF_GND -> RF_GND
- U2 pad 6: /channel1/RF_GND -> RF_GND
- U2 pad 7: /channel1/RF_GND -> RF_GND
- U2 pad 9: /channel1/RF_GND -> RF_GND
- U20 pad 10: /channel2/RESET -> /channel1/RESET
- U20 pad 11: /channel2/CLK -> /channel1/CLK
- U20 pad 13: /channel2/ENABLE -> /channel1/ENABLE
- U20 pad 14: /channel2/DIN -> /channel1/DOUT
- U20 pad 16: /channel2/5v -> 5v
- U20 pad 8: /channel2/DIG_GND -> DIG_GND
- U21 pad 3: /channel2/RF-In -> Net-(U21-RFC)
- U21 pad 4: /channel2/RF_GND -> RF_GND
- U21 pad 6: /channel2/RF_GND -> RF_GND
- U21 pad 7: /channel2/RF_GND -> RF_GND
- U21 pad 9: /channel2/RF_GND -> RF_GND
- U22 pad 4: /channel2/RF_GND -> RF_GND
- U22 pad 6: /channel2/RF_GND -> RF_GND
- U22 pad 7: /channel2/RF_GND -> RF_GND
- U22 pad 9: /channel2/RF_GND -> RF_GND
- U23 pad 4: /channel2/RF_GND -> RF_GND
- U23 pad 6: /channel2/RF_GND -> RF_GND
- U23 pad 7: /channel2/RF_GND -> RF_GND
- U23 pad 9: /channel2/RF_GND -> RF_GND
- U24 pad 4: /channel2/RF_GND -> RF_GND
- U24 pad 6: /channel2/RF_GND -> RF_GND
- U24 pad 7: /channel2/RF_GND -> RF_GND
- U24 pad 9: /channel2/RF_GND -> RF_GND
- U25 pad 1: /channel2/5v -> 5v
- U25 pad 11: /channel2/RF_GND -> RF_GND
- U25 pad 13: /channel2/RF_GND -> RF_GND
- U25 pad 15: /channel2/RF_GND -> RF_GND
- U25 pad 3: /channel2/5v -> 5v
- U25 pad 5: /channel2/5v -> 5v
- U25 pad 7: /channel2/5v -> 5v
- U25 pad 9: /channel2/RF_GND -> RF_GND
- U26 pad 4: /channel2/RF_GND -> RF_GND
- U26 pad 6: /channel2/RF_GND -> RF_GND
- U26 pad 7: /channel2/RF_GND -> RF_GND
- U26 pad 9: /channel2/RF_GND -> RF_GND
- U27 pad 4: /channel2/RF_GND -> RF_GND
- U27 pad 6: /channel2/RF_GND -> RF_GND
- U27 pad 7: /channel2/RF_GND -> RF_GND
- U27 pad 9: /channel2/RF_GND -> RF_GND
- U28 pad 4: /channel2/RF_GND -> RF_GND
- U28 pad 6: /channel2/RF_GND -> RF_GND
- U28 pad 7: /channel2/RF_GND -> RF_GND
- U28 pad 9: /channel2/RF_GND -> RF_GND
- U29 pad 4: /channel2/RF_GND -> RF_GND
- U29 pad 6: /channel2/RF_GND -> RF_GND
- U29 pad 7: /channel2/RF_GND -> RF_GND
- U29 pad 9: /channel2/RF_GND -> RF_GND
- U3 pad 4: /channel1/RF_GND -> RF_GND
- U3 pad 6: /channel1/RF_GND -> RF_GND
- U3 pad 7: /channel1/RF_GND -> RF_GND
- U3 pad 9: /channel1/RF_GND -> RF_GND
- U30 pad 1: /channel2/5v -> 5v
- U30 pad 11: /channel2/RF_GND -> RF_GND
- U30 pad 13: /channel2/RF_GND -> RF_GND
- U30 pad 15: /channel2/RF_GND -> RF_GND
- U30 pad 3: /channel2/5v -> 5v
- U30 pad 5: /channel2/5v -> 5v
- U30 pad 7: /channel2/5v -> 5v
- U30 pad 9: /channel2/RF_GND -> RF_GND
- U31 pad 4: /channel2/RF_GND -> RF_GND
- U31 pad 6: /channel2/RF_GND -> RF_GND
- U31 pad 7: /channel2/RF_GND -> RF_GND
- U31 pad 9: /channel2/RF_GND -> RF_GND
- U32 pad 4: /channel2/RF_GND -> RF_GND
- U32 pad 6: /channel2/RF_GND -> RF_GND
- U32 pad 7: /channel2/RF_GND -> RF_GND
- U32 pad 9: /channel2/RF_GND -> RF_GND
- U33 pad 4: /channel2/RF_GND -> RF_GND
- U33 pad 6: /channel2/RF_GND -> RF_GND
- U33 pad 7: /channel2/RF_GND -> RF_GND
- U33 pad 9: /channel2/RF_GND -> RF_GND
- U34 pad 4: /channel2/RF_GND -> RF_GND
- U34 pad 6: /channel2/RF_GND -> RF_GND
- U34 pad 7: /channel2/RF_GND -> RF_GND
- U34 pad 9: /channel2/RF_GND -> RF_GND
- U35 pad 4: /channel2/RF_GND -> RF_GND
- U35 pad 6: /channel2/RF_GND -> RF_GND
- U35 pad 7: /channel2/RF_GND -> RF_GND
- U35 pad 9: /channel2/RF_GND -> RF_GND
- U36 pad 4: /channel2/RF_GND -> RF_GND
- U36 pad 6: /channel2/RF_GND -> RF_GND
- U36 pad 7: /channel2/RF_GND -> RF_GND
- U36 pad 9: /channel2/RF_GND -> RF_GND
- U37 pad 4: /channel2/RF_GND -> RF_GND
- U37 pad 6: /channel2/RF_GND -> RF_GND
- U37 pad 7: /channel2/RF_GND -> RF_GND
- U37 pad 9: /channel2/RF_GND -> RF_GND
- U38 pad 3: Net-(U38-RFC) -> /channel2/RF-In
- U38 pad 4: /channel2/RF_GND -> RF_GND
- U38 pad 6: /channel2/RF_GND -> RF_GND
- U38 pad 7: /channel2/RF_GND -> RF_GND
- U38 pad 9: /channel2/RF_GND -> RF_GND
- U39 pad 10: /channel3/RESET -> /channel1/RESET
- U39 pad 11: /channel3/CLK -> /channel1/CLK
- U39 pad 13: /channel3/ENABLE -> /channel1/ENABLE
- U39 pad 14: /channel3/DIN -> /channel2/DOUT
- U39 pad 16: /channel3/5v -> 5v
- U39 pad 8: /channel3/DIG_GND -> DIG_GND
- U4 pad 4: /channel1/RF_GND -> RF_GND
- U4 pad 6: /channel1/RF_GND -> RF_GND
- U4 pad 7: /channel1/RF_GND -> RF_GND
- U4 pad 9: /channel1/RF_GND -> RF_GND
- U40 pad 3: /channel3/RF-In -> Net-(U40-RFC)
- U40 pad 4: /channel3/RF_GND -> RF_GND
- U40 pad 6: /channel3/RF_GND -> RF_GND
- U40 pad 7: /channel3/RF_GND -> RF_GND
- U40 pad 9: /channel3/RF_GND -> RF_GND
- U41 pad 4: /channel3/RF_GND -> RF_GND
- U41 pad 6: /channel3/RF_GND -> RF_GND
- U41 pad 7: /channel3/RF_GND -> RF_GND
- U41 pad 9: /channel3/RF_GND -> RF_GND
- U42 pad 4: /channel3/RF_GND -> RF_GND
- U42 pad 6: /channel3/RF_GND -> RF_GND
- U42 pad 7: /channel3/RF_GND -> RF_GND
- U42 pad 9: /channel3/RF_GND -> RF_GND
- U43 pad 4: /channel3/RF_GND -> RF_GND
- U43 pad 6: /channel3/RF_GND -> RF_GND
- U43 pad 7: /channel3/RF_GND -> RF_GND
- U43 pad 9: /channel3/RF_GND -> RF_GND
- U44 pad 1: /channel3/5v -> 5v
- U44 pad 11: /channel3/RF_GND -> RF_GND
- U44 pad 13: /channel3/RF_GND -> RF_GND
- U44 pad 15: /channel3/RF_GND -> RF_GND
- U44 pad 3: /channel3/5v -> 5v
- U44 pad 5: /channel3/5v -> 5v
- U44 pad 7: /channel3/5v -> 5v
- U44 pad 9: /channel3/RF_GND -> RF_GND
- U45 pad 4: /channel3/RF_GND -> RF_GND
- U45 pad 6: /channel3/RF_GND -> RF_GND
- U45 pad 7: /channel3/RF_GND -> RF_GND
- U45 pad 9: /channel3/RF_GND -> RF_GND
- U46 pad 4: /channel3/RF_GND -> RF_GND
- U46 pad 6: /channel3/RF_GND -> RF_GND
- U46 pad 7: /channel3/RF_GND -> RF_GND
- U46 pad 9: /channel3/RF_GND -> RF_GND
- U47 pad 4: /channel3/RF_GND -> RF_GND
- U47 pad 6: /channel3/RF_GND -> RF_GND
- U47 pad 7: /channel3/RF_GND -> RF_GND
- U47 pad 9: /channel3/RF_GND -> RF_GND
- U48 pad 4: /channel3/RF_GND -> RF_GND
- U48 pad 6: /channel3/RF_GND -> RF_GND
- U48 pad 7: /channel3/RF_GND -> RF_GND
- U48 pad 9: /channel3/RF_GND -> RF_GND
- U49 pad 1: /channel3/5v -> 5v
- U49 pad 11: /channel3/RF_GND -> RF_GND
- U49 pad 13: /channel3/RF_GND -> RF_GND
- U49 pad 15: /channel3/RF_GND -> RF_GND
- U49 pad 3: /channel3/5v -> 5v
- U49 pad 5: /channel3/5v -> 5v
- U49 pad 7: /channel3/5v -> 5v
- U49 pad 9: /channel3/RF_GND -> RF_GND
- U5 pad 4: /channel1/RF_GND -> RF_GND
- U5 pad 6: /channel1/RF_GND -> RF_GND
- U5 pad 7: /channel1/RF_GND -> RF_GND
- U5 pad 9: /channel1/RF_GND -> RF_GND
- U50 pad 4: /channel3/RF_GND -> RF_GND
- U50 pad 6: /channel3/RF_GND -> RF_GND
- U50 pad 7: /channel3/RF_GND -> RF_GND
- U50 pad 9: /channel3/RF_GND -> RF_GND
- U51 pad 4: /channel3/RF_GND -> RF_GND
- U51 pad 6: /channel3/RF_GND -> RF_GND
- U51 pad 7: /channel3/RF_GND -> RF_GND
- U51 pad 9: /channel3/RF_GND -> RF_GND
- U52 pad 4: /channel3/RF_GND -> RF_GND
- U52 pad 6: /channel3/RF_GND -> RF_GND
- U52 pad 7: /channel3/RF_GND -> RF_GND
- U52 pad 9: /channel3/RF_GND -> RF_GND
- U53 pad 4: /channel3/RF_GND -> RF_GND
- U53 pad 6: /channel3/RF_GND -> RF_GND
- U53 pad 7: /channel3/RF_GND -> RF_GND
- U53 pad 9: /channel3/RF_GND -> RF_GND
- U54 pad 4: /channel3/RF_GND -> RF_GND
- U54 pad 6: /channel3/RF_GND -> RF_GND
- U54 pad 7: /channel3/RF_GND -> RF_GND
- U54 pad 9: /channel3/RF_GND -> RF_GND
- U55 pad 4: /channel3/RF_GND -> RF_GND
- U55 pad 6: /channel3/RF_GND -> RF_GND
- U55 pad 7: /channel3/RF_GND -> RF_GND
- U55 pad 9: /channel3/RF_GND -> RF_GND
- U56 pad 4: /channel3/RF_GND -> RF_GND
- U56 pad 6: /channel3/RF_GND -> RF_GND
- U56 pad 7: /channel3/RF_GND -> RF_GND
- U56 pad 9: /channel3/RF_GND -> RF_GND
- U57 pad 3: Net-(U57-RFC) -> /channel3/RF-In
- U57 pad 4: /channel3/RF_GND -> RF_GND
- U57 pad 6: /channel3/RF_GND -> RF_GND
- U57 pad 7: /channel3/RF_GND -> RF_GND
- U57 pad 9: /channel3/RF_GND -> RF_GND
- U6 pad 4: /channel1/RF_GND -> RF_GND
- U6 pad 6: /channel1/RF_GND -> RF_GND
- U6 pad 7: /channel1/RF_GND -> RF_GND
- U6 pad 9: /channel1/RF_GND -> RF_GND
- U7 pad 4: /channel1/RF_GND -> RF_GND
- U7 pad 6: /channel1/RF_GND -> RF_GND
- U7 pad 7: /channel1/RF_GND -> RF_GND
- U7 pad 9: /channel1/RF_GND -> RF_GND
- U8 pad 4: /channel1/RF_GND -> RF_GND
- U8 pad 6: /channel1/RF_GND -> RF_GND
- U8 pad 7: /channel1/RF_GND -> RF_GND
- U8 pad 9: /channel1/RF_GND -> RF_GND
- U9 pad 4: /channel1/RF_GND -> RF_GND
- U9 pad 6: /channel1/RF_GND -> RF_GND
- U9 pad 7: /channel1/RF_GND -> RF_GND
- U9 pad 9: /channel1/RF_GND -> RF_GND
Routing:
- net RF_GND: track 0.00 -> 753.2 mm, vias 0 -> 525
- net 5v: track 0.00 -> 440.6 mm
- net DIG_GND: track 0.00 -> 408.7 mm, vias 0 -> 36
- net /channel1/RF_GND: track 199.7 -> 0.00 mm, vias 177 -> 0
- net /channel3/RF_GND: track 199.7 -> 0.00 mm, vias 177 -> 0
- net /channel2/RF_GND: track 199.7 -> 0.00 mm, vias 177 -> 0
- net Net-(U57-RFC): track 192.3 -> 0.00 mm
- net Net-(U16-RFC): track 192.3 -> 0.00 mm
- net Net-(U38-RFC): track 192.3 -> 0.00 mm
- net /channel3/5v: track 146.9 -> 0.00 mm
- net /channel1/5v: track 146.9 -> 0.00 mm
- net /channel2/5v: track 146.9 -> 0.00 mm
- net /channel3/DIG_GND: track 136.2 -> 0.00 mm, vias 12 -> 0
- net /channel2/DIG_GND: track 136.2 -> 0.00 mm, vias 12 -> 0
- net /channel1/DIG_GND: track 136.2 -> 0.00 mm, vias 12 -> 0
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- added copper zone on B.Cu, net 5v
- removed copper zone on B.Cu, net /channel1/5v
- removed copper zone on F.Cu, net /channel1/RF_GND
- removed copper zone on B.Cu, net /channel2/5v
- removed copper zone on F.Cu, net /channel2/RF_GND
- removed copper zone on B.Cu, net /channel3/5v
- removed copper zone on F.Cu, net /channel3/RF_GND
Other:
- board size 240 x 177.2 mm -> 249.9 x 160.1 mm
- board text removed: "East"
- board text removed: "North"
- board text removed: "West"

Commit message: Finalized simulation PCB.
Parts:
- added C7: 470n, Capacitor_THT:C_Radial_D10.0mm_H12.5mm_P5.00mm, F.Cu at (222.0, 44.4)
- added C8: 22uF, Capacitor_THT:CP_Radial_D6.3mm_P2.50mm, F.Cu at (231.8, 40.1)
- added FB4: FerriteBead, Inductor_SMD:L_0805_2012Metric_Pad1.05x1.20mm_HandSolder, F.Cu at (202.9, 37.1)
- added J6: Conn_01x02, Connector_PinHeader_2.54mm:PinHeader_1x02_P2.54mm_Vertical, F.Cu at (240.8, 39.9)
- added REF**: MountingHole_4.3mm_M4, MountingHole:MountingHole_4.3mm_M4, F.Cu at (32.8, 150.4)
- added REF**: MountingHole_4.3mm_M4, MountingHole:MountingHole_4.3mm_M4, F.Cu at (254.5, 89.1)
- added REF**: MountingHole_4.3mm_M4, MountingHole:MountingHole_4.3mm_M4, F.Cu at (32.8, 61.1)
- added REF**: MountingHole_4.3mm_M4, MountingHole:MountingHole_4.3mm_M4, F.Cu at (259.5, 183.6)
- added U58: LM78M05_TO220, Package_TO_SOT_THT:TO-220-3_Vertical, F.Cu at (216.5, 37.9)
- R130: moved to B.Cu
- moved R130 76.4 mm to (263.8, 45.4), turned to 180 degrees
- moved J4 63.1 mm to (260.3, 38.3), turned to -90 degrees
- moved R132 10.7 mm to (46.8, 37.9)
- moved R133 10.4 mm to (47.5, 49.1)
- moved R131 10.3 mm to (51.2, 43.9)
Connections:
- J4 pad 1: VCC -> 5v
- J4 pad 2: /channel2/DOUT -> /channel1/DIN
- J4 pad 8: unconnected-(J4-Pin_8-Pad8) -> /channel1/RESET
- J5 pad 2: unconnected-(J5-Ext-Pad2) -> RF_GND
- R130 pad 1: VCC -> 5v
Routing:
- net /channel1/RF-In: track 0.00 -> 283.1 mm
- net /channel3/RF-In: track 0.00 -> 282.6 mm
- net /channel2/RF-In: track 0.00 -> 282.2 mm
- net /channel1/RCLK: track 0.00 -> 153.8 mm
- net /channel1/RESET: track 0.00 -> 147.6 mm, vias 0 -> 3
- net /channel1/ENABLE: track 0.00 -> 142.3 mm, vias 0 -> 4
- net /channel1/CLK: track 0.00 -> 142.2 mm, vias 0 -> 3
- net /channel1/DIN: track 0.00 -> 139.7 mm, vias 0 -> 1
- net /channel2/RCLK: track 0.00 -> 104.3 mm, vias 0 -> 1
- net /channel3/RCLK: track 0.00 -> 52.8 mm, vias 0 -> 1
- net /channel1/DOUT: track 0.00 -> 47.9 mm
- net /channel2/DOUT: track 0.00 -> 47.7 mm
- net RF_GND: track 753.2 -> 791.7 mm, vias 525 -> 744
- net Net-(J6-Pin_1): track 0.00 -> 36.5 mm
- net Net-(J5-In): track 16.5 -> 41.8 mm
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- added copper zone on In2.Cu, net DIG_GND
- added copper zone on F.Cu, net RF_GND
- added copper zone on In1.Cu, net RF_GND
Other:
- board text added: "5v"
- board text added: "9v"
- board text added: "CLK"
- board text added: "DIN"
- board text added: "Direction simulator"
- board text added: "E"
- board text added: "EN"
- board text added: "East"
- board text added: "GND"
- board text added: "Input"
- board text added: "N"
- board text added: "North"
- board text added: "RES"
- board text added: "W"
- board text added: "West"

Commit message: Added gerber files.
Parts:
- added R134: 24.9, Resistor_SMD:R_0805_2012Metric_Pad1.20x1.40mm_HandSolder, F.Cu at (37.4, 44.0)
- U58: value LM78M05_TO220 -> LM2940CT-5.0
- moved REF** 52.2 mm to (271.8, 39.8)
- moved REF** 13.4 mm to (271.4, 189.7)
- moved R131 0.25 mm to (51.2, 44.1)
Connections:
- R131 pad 1: Net-(J5-In) -> Net-(R131-Pad1)
- R132 pad 1: Net-(J5-In) -> Net-(R131-Pad1)
- R133 pad 1: Net-(J5-In) -> Net-(R131-Pad1)
Routing:
- net Net-(J5-In): track 41.8 -> 7.04 mm
- net Net-(R131-Pad1): track 0.00 -> 32.9 mm
- net /channel1/RCLK: track 153.8 -> 146.7 mm
- net /channel2/RCLK: track 104.3 -> 97.7 mm
- net /channel1/DIN: track 139.7 -> 137.4 mm
