File: spi_amp/spi-amp/spi-amp.kicad_sch (KiCad schematic)
At the start: 27 parts, among them J1 IN+, J2 IN-, J3 OUT+, J4 OUT-, J5 Conn_01x06, U1 LMH6401, U2 LM78M05_TO220

Commit message: Finalized SPI interface PCB
Parts:
- H1, H2: footprint MountingHole:MountingHole_2.7mm_M2.5_Pad -> MountingHole:MountingHole_3.2mm_M3_Pad
Changed lines of the file:
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@@
 			)
 		)
-		(property "Footprint" "MountingHole:MountingHole_2.7mm_M2.5_Pad"
+		(property "Footprint" "MountingHole:MountingHole_3.2mm_M3_Pad"
 			(at 149.86 128.27 0)
 			(hide yes)
@@
 			)
 		)
-		(property "Footprint" "MountingHole:MountingHole_2.7mm_M2.5_Pad"
+		(property "Footprint" "MountingHole:MountingHole_3.2mm_M3_Pad"
 			(at 176.53 128.27 0)
 			(hide yes)
