File: spi_amp/spi-amp/spi-amp.kicad_pcb (KiCad board)
At the start: 4 copper layers, 28.7 x 66.1 mm, 27 parts, among them J1 IN+, J2 IN-, J3 OUT+, J4 OUT-, J5 Conn_01x06, U1 LMH6401, U2 LM78M05_TO220

Commit message: Fixed spi-amp DRC problems.
Routing:
- net Net-(R2-Pad1): track 4.25 -> 5.03 mm
- net Net-(R1-Pad1): track 4.34 -> 5.02 mm
- net DIG_GND: vias 141 -> 138
