File: spiband/spiband/spiband.kicad_pcb (KiCad board)
At the start: 4 copper layers, 66.2 x 41.6 mm, 50 parts, among them J1 RJ45_Shielded, J2 Conn_01x06, J3 Conn_01x06, J4 Conn_01x06, J5 Conn_01x02, J6 Screw_Terminal_01x02, U1 MAX3485, U10 SN74LVC1T45DBV, U11 LM1086CT-3.3, U2 MAX3485, U3 MAX3485, U4 MAX3232, U5 74HC04, U6 TLV70018_SOT353, U7 SN74HC153DR1G4, U8 SN74LVC1T45DBV, U9 SN74LVC1T45DBV

Commit message: Finalized the PCBs and sent them to review.
Routing:
- net GND: vias 60 -> 85
Changed lines of the file:
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@@
+	)
+	(via
+		(at 209.55 92.65)
+		(size 0.6)
+		(drill 0.3)
+		(layers "F.Cu" "B.Cu")
+		(free yes)
+		(net "GND")
 	)
 	(via
@@
 	)
 	(via
-		(at 172.4 102.8)
+		(at 168.1 102.55)
 		(size 0.6)
 		(drill 0.3)
@@
 	)
 	(via
+		(at 165.15 84.6)
+		(size 0.6)
+		(drill 0.3)
+		(layers "F.Cu" "B.Cu")
+		(free yes)
+		(net "GND")
+	)
+	(via
+		(at 210.7 84.7)
+		(size 0.6)
+		(drill 0.3)
+		(layers "F.Cu" "B.Cu")
+		(free yes)
+		(net "GND")
+	)
+	(via
 		(at 150.2 86.5)
 		(size 0.6)
@@
 	)
 	(via
+		(at 164.55 96.1)
+		(size 0.6)
+		(drill 0.3)
+		(layers "F.Cu" "B.Cu")
+		(free yes)
+		(net "GND")
+	)
+	(via
+		(at 171.7 89.5)
+		(size 0.6)
+		(drill 0.3)
+		(layers "F.Cu" "B.Cu")
+		(free yes)
+		(net "GND")
+	)
+	(via
 		(at 210.6 100.3)
 		(size 0.6)
@@
 	)
 	(via
+		(at 172.6 110.95)
+		(size 0.6)
+		(drill 0.3)
+		(layers "F.Cu" "B.Cu")
+		(free yes)
+		(net "GND")
+	)
+	(via
 		(at 185.2 112.7)
 		(size 0.6)
@@
 	)
 	(via
+		(at 164.2 93.85)
+		(size 0.6)
+		(drill 0.3)
+		(layers "F.Cu" "B.Cu")
+		(free yes)
+		(net "GND")
+	)
+	(via
+		(at 171.75 93.05)
+		(size 0.6)
+		(drill 0.3)
+		(layers "F.Cu" "B.Cu")
+		(free yes)
+		(net "GND")
+	)
+	(via
 		(at 176.4 111)
 		(size 0.6)
@@
 	)
 	(via
+		(at 212.75 124.55)
+		(size 0.6)
+		(drill 0.3)
+		(layers "F.Cu" "B.Cu")
+		(free yes)
+		(net "GND")
+	)
+	(via
+		(at 172.6 112.35)
+		(size 0.6)
+		(drill 0.3)
+		(layers "F.Cu" "B.Cu")
+		(free yes)
+		(net "GND")
+	)
+	(via
 		(at 176.2 88)
 		(size 0.6)
@@
 	)
 	(via
+		(at 173.3 105.85)
+		(size 0.6)
+		(drill 0.3)
+		(layers "F.Cu" "B.Cu")
+		(free yes)
+		(net "GND")
+	)
+	(via
+		(at 171.6 103.2)
+		(size 0.6)
+		(drill 0.3)
+		(layers "F.Cu" "B.Cu")
+		(free yes)
+		(net "GND")
+	)
+	(via
 		(at 188.6 98.6)
 		(size 0.6)
@@
 	)
 	(via
+		(at 171.4 102.15)
+		(size 0.6)
+		(drill 0.3)
+		(layers "F.Cu" "B.Cu")
+		(free yes)
+		(net "GND")
+	)
+	(via
 		(at 183.6 114.2)
 		(size 0.6)
@@
 	)
 	(via
+		(at 168 91.15)
+		(size 0.6)
+		(drill 0.3)
+		(layers "F.Cu" "B.Cu")
+		(free yes)
+		(net "GND")
+	)
+	(via
+		(at 176.05 112.2)
+		(size 0.6)
+		(drill 0.3)
+		(layers "F.Cu" "B.Cu")
+		(free yes)
+		(net "GND")
+	)
+	(via
 		(at 167.6 119.3)
 		(size 0.6)
@@
 	)
 	(via
+		(at 175.7 108.9)
+		(size 0.6)
+		(drill 0.3)
+		(layers "F.Cu" "B.Cu")
+		(free yes)
+		(net "GND")
+	)
+	(via
 		(at 208.4 98.6)
 		(size 0.6)
@@
 	)
 	(via
+		(at 210.15 95.4)
+		(size 0.6)
+		(drill 0.3)
+		(layers "F.Cu" "B.Cu")
+		(free yes)
+		(net "GND")
+	)
+	(via
+		(at 168.2 92.45)
+		(size 0.6)
+		(drill 0.3)
+		(layers "F.Cu" "B.Cu")
+		(free yes)
+		(net "GND")
+	)
+	(via
 		(at 163.6 86.8)
 		(size 0.6)
@@
 	)
 	(via
-		(at 176.9 104)
-		(size 0.6)
-		(drill 0.3)
-		(layers "F.Cu" "B.Cu")
-		(free yes)
-		(net "GND")
-	)
-	(via
 		(at 196.7 98.9)
 		(size 0.6)
@@
 	)
 	(via
-		(at 171.7 109.7)
+		(at 176.5 105.3)
+		(size 0.6)
+		(drill 0.3)
+		(layers "F.Cu" "B.Cu")
+		(free yes)
+		(net "GND")
+	)
+	(via
+		(at 172.6 109.7)
 		(size 0.6)
 		(drill 0.3)
@@
 	)
 	(via
+		(at 176.55 104.15)
+		(size 0.6)
+		(drill 0.3)
+		(layers "F.Cu" "B.Cu")
+		(free yes)
+		(net "GND")
+	)
+	(via
 		(at 209.8 123.5)
 		(size 0.6)
@@
 	)
 	(via
+		(at 165.15 85.55)
+		(size 0.6)
+		(drill 0.3)
+		(layers "F.Cu" "B.Cu")
+		(free yes)
+		(net "GND")
+	)
+	(via
 		(at 170 87.9725)
 		(size 0.6)
@@
 	)
 	(via
+		(at 208.2 85.4)
+		(size 0.6)
+		(drill 0.3)
+		(layers "F.Cu" "B.Cu")
+		(free yes)
+		(net "GND")
+	)
+	(via
 		(at 170 101.5)
 		(size 0.6)
@@
 	)
 	(via
+		(at 208.25 94.1)
+		(size 0.6)
+		(drill 0.3)
+		(layers "F.Cu" "B.Cu")
+		(free yes)
+		(net "GND")
+	)
+	(via
 		(at 181.9 112.8)
 		(size 0.6)
@@
 	)
 	(via
+		(at 176.5 102.55)
+		(size 0.6)
+		(drill 0.3)
+		(layers "F.Cu" "B.Cu")
+		(free yes)
+		(net "GND")
+	)
+	(via
+		(at 212.75 122.5)
+		(size 0.6)
+		(drill 0.3)
+		(layers "F.Cu" "B.Cu")
+		(free yes)
+		(net "GND")
+	)
+	(via
 		(at 176.4 84.6)
 		(size 0.6)
@@
 		(size 0.6)
 		(drill 0.3)
+		(layers "F.Cu" "B.Cu")
+		(free yes)
+		(net "GND")
+	)
+	(via
+		(at 169.05 89.45)
+		(size 0.6)
+		(drill 0.3)
